Commit message: refactor: disabled topplate and all sensor(incomplete)

File: husky_description/urdf/decorations.urdf.xacro (robot description, xacro)
@@ -45,5 +45,5 @@
     <!-- Top Plate -->
     <xacro:property name="pacs_enable"                  value="$(optenv HUSKY_PACS_ENABLED false)"/>
-    <xacro:property name="top_plate_enable"             value="$(optenv HUSKY_TOP_PLATE_ENABLED true)"/>
+    <xacro:property name="top_plate_enable"             value="$(optenv HUSKY_TOP_PLATE_ENABLED false)"/>
     <xacro:property name="large_top_plate_enable"       value="$(optenv HUSKY_LARGE_TOP_PLATE false)"/>
     <xacro:property name="user_rail_enable"             value="$(optenv HUSKY_USER_RAIL_ENABLED true)"/>

File: husky_description/urdf/husky.urdf.xacro (robot description, xacro)
@@ -79,5 +79,5 @@
   <xacro:property name="realsense_model"          value="$(arg realsense_model)"/>
   <!-- Realsense Camera New -->
-  <xacro:arg name="realsense_enabled_new"             default="$(optenv HUSKY_REALSENSE_ENABLED 1)" />
+  <xacro:arg name="realsense_enabled_new"             default="$(optenv HUSKY_REALSENSE_ENABLED 0)" />
   <xacro:arg name="realsense_mode_new"               default="$(optenv HUSKY_REALSENSE_MODEL d435)"/>
   <xacro:arg name="realsense_topic_new"               default="$(optenv HUSKY_REALSENSE_TOPIC realsense)" />
@@ -123,5 +123,5 @@
   <xacro:arg name="cpr_urdf_extras" default="$(optenv CPR_URDF_EXTRAS empty.urdf)" />
   <!-- OutdoorNav -->
-  <xacro:arg name="outdoornav_enabled"       default="$(optenv OUTDOORNAV_ENABLED 1)" />
+  <xacro:arg name="outdoornav_enabled"       default="$(optenv OUTDOORNAV_ENABLED 0)" />
   <xacro:arg name="outdoornav_configuration" default="$(optenv OUTDOORNAV_CONFIGURATION standard)" />
   <!-- Included URDF/XACRO Files -->
@@ -130,8 +130,9 @@
   <!-- <xacro:include filename="$(find husky_description)/urdf/accessories/sick_lms1xx_mount.urdf.xacro"/> -->
   <!-- <xacro:include filename="$(find husky_description)/urdf/accessories/flir_blackfly_mount.urdf.xacro"/> -->
-  <xacro:include filename="$(find husky_description)/urdf/accessories/sensor_arch.urdf.xacro"/>
-  <xacro:include filename="$(find husky_description)/urdf/accessories/vlp16_mount.urdf.xacro"/>
+  <!-- <xacro:include filename="$(find husky_description)/urdf/accessories/sensor_arch.urdf.xacro"/> -->
+  <!-- <xacro:include filename="$(find husky_description)/urdf/accessories/vlp16_mount.urdf.xacro"/> -->
   <xacro:include filename="$(find husky_description)/urdf/decorations.urdf.xacro" />
   <xacro:include filename="$(find husky_description)/urdf/wheel.urdf.xacro" />
+  <xacro:include filename="$(find cpr_onav_description)/urdf/husky_observer.urdf.xacro" />
   <xacro:property name="M_PI" value="3.14159"/>
   <!-- Base Size -->
