Commit message: fix: realsense camera urdf errors (not fixed)

File: husky_description/urdf/husky.urdf.xacro (robot description, xacro)
@@ -70,5 +70,5 @@
   <xacro:arg name="laser_3d_secondary_rpy"        default="$(optenv HUSKY_LASER_3D_SECONDARY_RPY 0 0 -3.14159)" />
   <!-- Realsense Camera Primary and Secondary -->
-  <xacro:arg name="realsense_enabled"             default="$(optenv HUSKY_REALSENSE_ENABLED 1)" />
+  <xacro:arg name="realsense_enabled"             default="$(optenv HUSKY_REALSENSE_ENABLED 0)" />
   <xacro:arg name="realsense_model"               default="$(optenv HUSKY_REALSENSE_MODEL d435)"/>
   <xacro:arg name="realsense_topic"               default="$(optenv HUSKY_REALSENSE_TOPIC realsense)" />
@@ -77,4 +77,13 @@
   <xacro:arg name="realsense_xyz"                 default="$(optenv HUSKY_REALSENSE_XYZ 0.35 0 0.01)" />
   <xacro:arg name="realsense_rpy"                 default="$(optenv HUSKY_REALSENSE_RPY 0 0 0)" />
+  <xacro:property name="realsense_model"          value="$(arg realsense_model)"/>
+  <!-- Realsense Camera New -->
+  <xacro:arg name="realsense_enabled_new"             default="$(optenv HUSKY_REALSENSE_ENABLED 1)" />
+  <xacro:arg name="realsense_mode_new"               default="$(optenv HUSKY_REALSENSE_MODEL d435)"/>
+  <xacro:arg name="realsense_topic_new"               default="$(optenv HUSKY_REALSENSE_TOPIC realsense)" />
+  <xacro:arg name="realsense_prefix_new"              default="$(optenv HUSKY_REALSENSE_PREFIX camera)" />
+  <xacro:arg name="realsense_parent_new"              default="$(optenv HUSKY_REALSENSE_PARENT top_plate_link)" />
+  <xacro:arg name="realsense_xyz_new"                 default="$(optenv HUSKY_REALSENSE_XYZ 0.35 0 0.01)" />
+  <xacro:arg name="realsense_rpy_new"                 default="$(optenv HUSKY_REALSENSE_RPY 0 0 0)" />
   <xacro:property name="realsense_model"          value="$(arg realsense_model)"/>
   <xacro:arg name="realsense_secondary_enabled"   default="$(optenv HUSKY_REALSENSE_SECONDARY_ENABLED 0)" />
@@ -117,10 +126,11 @@
   <xacro:arg name="outdoornav_configuration" default="$(optenv OUTDOORNAV_CONFIGURATION standard)" />
   <!-- Included URDF/XACRO Files -->
-  <xacro:include filename="$(find husky_description)/urdf/accessories/hokuyo_ust10.urdf.xacro" />
-  <xacro:include filename="$(find husky_description)/urdf/accessories/intel_realsense.urdf.xacro"/>
-  <xacro:include filename="$(find husky_description)/urdf/accessories/flir_blackfly_mount.urdf.xacro"/>
+  <!-- <xacro:include filename="$(find husky_description)/urdf/accessories/hokuyo_ust10.urdf.xacro" /> -->
+  <!-- <xacro:include filename="$(find husky_description)/urdf/accessories/intel_realsense.urdf.xacro"/> -->
+  <!-- <xacro:include filename="$(find husky_description)/urdf/accessories/sick_lms1xx_mount.urdf.xacro"/> -->
+  <!-- <xacro:include filename="$(find husky_description)/urdf/accessories/flir_blackfly_mount.urdf.xacro"/> -->
   <xacro:include filename="$(find husky_description)/urdf/accessories/sensor_arch.urdf.xacro"/>
-  <!-- <xacro:include filename="$(find husky_description)/urdf/accessories/sick_lms1xx_mount.urdf.xacro"/> -->
   <xacro:include filename="$(find husky_description)/urdf/accessories/vlp16_mount.urdf.xacro"/>
+  <!-- <xacro:include filename="$(find realsense2_description)/urdf/_d435.urdf.xacro" /> -->
   <xacro:include filename="$(find husky_description)/urdf/decorations.urdf.xacro" />
   <xacro:include filename="$(find husky_description)/urdf/wheel.urdf.xacro" />
@@ -274,4 +284,25 @@
     </xacro:realsense_sensor>
   </xacro:if>
+  <!-- Intel Realsense New-->
+  <xacro:if value="$(arg realsense_enabled_new)">
+    <!-- Include the correct model based on realsense_mode_new -->
+    <xacro:include filename="$(find realsense2_description)/urdf/_$(arg realsense_mode_new).urdf.xacro" />
+    <!-- Define the camera link -->
+    <link name="realsense_camera_link" />
+    <!-- Use the included sensor macro -->
+    <xacro:sensor_d435
+          name="$(arg realsense_prefix_new)"
+          topics_ns="$(arg realsense_topic_new)"
+          parent="realsense_camera_link"
+          publish_pointcloud="true">
+      <origin xyz="0 0 0" rpy="0 0 0" />
+    </xacro:sensor_d435>
+    <!-- Mount joint (position and orientation come from args) -->
+    <joint name="${arg realsense_prefix_new}_mount" type="fixed">
+        <origin xyz="$(arg realsense_xyz_new)" rpy="$(arg realsense_rpy_new)"/>
+        <parent link="$(arg realsense_parent_new)"/>
+        <child link="realsense_camera_link"/>
+    </joint>
+  </xacro:if>
   <!-- BlackflyS Camera Primary and Secondary -->
   <xacro:if value="$(arg blackfly_enabled)">

Commit message: feat: added new realsesne2 description v3.1.7 with gazebo plugin fix: mod husky urdf to import new realsense

File: husky_description/urdf/husky.urdf.xacro (robot description, xacro)
@@ -82,5 +82,5 @@
   <xacro:arg name="realsense_mode_new"               default="$(optenv HUSKY_REALSENSE_MODEL d435)"/>
   <xacro:arg name="realsense_topic_new"               default="$(optenv HUSKY_REALSENSE_TOPIC realsense)" />
-  <xacro:arg name="realsense_prefix_new"              default="$(optenv HUSKY_REALSENSE_PREFIX camera)" />
+  <xacro:arg name="realsense_prefix_new"              default="$(optenv HUSKY_REALSENSE_PREFIX realsense_camera)" />
   <xacro:arg name="realsense_parent_new"              default="$(optenv HUSKY_REALSENSE_PARENT top_plate_link)" />
   <xacro:arg name="realsense_xyz_new"                 default="$(optenv HUSKY_REALSENSE_XYZ 0.35 0 0.01)" />
@@ -97,5 +97,5 @@
   <!-- BlackflyS Camera Primary and Secondary -->
   <xacro:arg name="blackfly_enabled"                  default="$(optenv HUSKY_BLACKFLY 0)"/>
-  <xacro:arg name="blackfly_mount_enabled"            default="$(optenv HUSKY_BLACKFLY_MOUNT_ENABLED 1)"/>
+  <xacro:arg name="blackfly_mount_enabled"            default="$(optenv HUSKY_BLACKFLY_MOUNT_ENABLED 0)"/>
   <xacro:arg name="blackfly_mount_angle"              default="$(optenv HUSKY_BLACKFLY_MOUNT_ANGLE 0)"/>
   <xacro:arg name="blackfly_prefix"                   default="$(optenv HUSKY_BLACKFLY_PREFIX blackfly)"/>
@@ -104,5 +104,5 @@
   <xacro:arg name="blackfly_rpy"                      default="$(optenv HUSKY_BLACKFLY_RPY 0 0 0)"/>
   <xacro:arg name="blackfly_secondary_enabled"        default="$(optenv HUSKY_BLACKFLY_SECONDARY 0)"/>
-  <xacro:arg name="blackfly_secondary_mount_enabled"  default="$(optenv HUSKY_BLACKFLY_SECONDARY_MOUNT_ENABLED 1)"/>
+  <xacro:arg name="blackfly_secondary_mount_enabled"  default="$(optenv HUSKY_BLACKFLY_SECONDARY_MOUNT_ENABLED 0)"/>
   <xacro:arg name="blackfly_secondary_mount_angle"    default="$(optenv HUSKY_BLACKFLY_SECONDARY_MOUNT_ANGLE 0)"/>
   <xacro:arg name="blackfly_secondary_prefix"         default="$(optenv HUSKY_BLACKFLY_SECONDARY_PREFIX blackfly_secondary)"/>
@@ -132,5 +132,4 @@
   <xacro:include filename="$(find husky_description)/urdf/accessories/sensor_arch.urdf.xacro"/>
   <xacro:include filename="$(find husky_description)/urdf/accessories/vlp16_mount.urdf.xacro"/>
-  <!-- <xacro:include filename="$(find realsense2_description)/urdf/_d435.urdf.xacro" /> -->
   <xacro:include filename="$(find husky_description)/urdf/decorations.urdf.xacro" />
   <xacro:include filename="$(find husky_description)/urdf/wheel.urdf.xacro" />
@@ -249,6 +248,7 @@
       </xacro:hokuyo_ust10_mount>
   </xacro:if>
+  <!-- ################# THIS IS OLD VERSION IMPORT ############################################################################# -->
   <!-- Intel Realsense Primary and Secondary -->
-  <xacro:property name="realsense_enabled" value="$(arg realsense_enabled)"/>
+  <!-- <xacro:property name="realsense_enabled" value="$(arg realsense_enabled)"/>
   <xacro:property name="realsense_secondary_enabled" value="$(arg realsense_secondary_enabled)"/>
   <xacro:if value="${realsense_enabled or realsense_secondary_enabled}">
@@ -283,24 +283,20 @@
       <origin xyz="$(arg realsense_secondary_xyz)" rpy="$(arg realsense_secondary_rpy)"/>
     </xacro:realsense_sensor>
-  </xacro:if>
+  </xacro:if> -->
+  <!-- ######################################################################################################################### -->
   <!-- Intel Realsense New-->
   <xacro:if value="$(arg realsense_enabled_new)">
     <!-- Include the correct model based on realsense_mode_new -->
+    <!-- Define the camera link -->
     <xacro:include filename="$(find realsense2_description)/urdf/_$(arg realsense_mode_new).urdf.xacro" />
-    <!-- Define the camera link -->
-    <link name="realsense_camera_link" />
-    <!-- Use the included sensor macro -->
-    <xacro:sensor_d435
-          name="$(arg realsense_prefix_new)"
-          topics_ns="$(arg realsense_topic_new)"
-          parent="realsense_camera_link"
-          publish_pointcloud="true">
-      <origin xyz="0 0 0" rpy="0 0 0" />
+    <link name="$(arg realsense_prefix_new)_link" />
+    <xacro:sensor_d435 name="camera" topics_ns="camera" parent="$(arg realsense_prefix_new)_link" publish_pointcloud="true">
+        <origin xyz="0 0 0" rpy="0 0 0" />
     </xacro:sensor_d435>
     <!-- Mount joint (position and orientation come from args) -->
-    <joint name="${arg realsense_prefix_new}_mount" type="fixed">
+    <joint name="$(arg realsense_prefix_new)_mount" type="fixed">
         <origin xyz="$(arg realsense_xyz_new)" rpy="$(arg realsense_rpy_new)"/>
         <parent link="$(arg realsense_parent_new)"/>
-        <child link="realsense_camera_link"/>
+        <child link="$(arg realsense_prefix_new)_link"/>
     </joint>
   </xacro:if>

Commit message: feat: added gps antenas left and right, realse camera and lidar added msg:(now the cpr_onav package not used just urdf copied to description package and used from there)

File: husky_description/urdf/husky.urdf.xacro (robot description, xacro)
@@ -55,5 +55,5 @@
   <xacro:arg name="laser_ust10_rear_rpy"      default="$(optenv HUSKY_UST10_SECONDARY_RPY 0 0 3.14159)" />
   <!-- Velodyne LiDAR Primary and Secondary -->
-  <xacro:arg name="laser_3d_enabled"              default="$(optenv HUSKY_LASER_3D_ENABLED 0)" />
+  <!-- <xacro:arg name="laser_3d_enabled"              default="$(optenv HUSKY_LASER_3D_ENABLED 0)" />
   <xacro:arg name="laser_3d_topic"                default="$(optenv HUSKY_LASER_3D_TOPIC points)"/>
   <xacro:arg name="laser_3d_tower"                default="$(optenv HUSKY_LASER_3D_TOWER 1)"/>
@@ -61,4 +61,12 @@
   <xacro:arg name="laser_3d_parent"               default="$(optenv HUSKY_LASER_3D_PARENT top_plate_link)"/>
   <xacro:arg name="laser_3d_xyz"                  default="$(optenv HUSKY_LASER_3D_XYZ 0 0 0)" />
+  <xacro:arg name="laser_3d_rpy"                  default="$(optenv HUSKY_LASER_3D_RPY 0 0 0)" /> -->
+  <!-- Velodyne LiDAR Primary and Secondary -->
+  <xacro:arg name="laser_3d_enabled"              default="$(optenv HUSKY_LASER_3D_ENABLED 1)" />
+  <xacro:arg name="laser_3d_topic"                default="$(optenv HUSKY_LASER_3D_TOPIC points)"/>
+  <xacro:arg name="laser_3d_tower"                default="$(optenv HUSKY_LASER_3D_TOWER 0)"/>
+  <xacro:arg name="laser_3d_prefix"               default="$(optenv HUSKY_LASER_3D_PREFIX )"/>
+  <xacro:arg name="laser_3d_parent"               default="$(optenv HUSKY_LASER_3D_PARENT backpack_link)"/>
+  <xacro:arg name="laser_3d_xyz"                  default="$(optenv HUSKY_LASER_3D_XYZ 0 0 0.26)" />
   <xacro:arg name="laser_3d_rpy"                  default="$(optenv HUSKY_LASER_3D_RPY 0 0 0)" />
   <xacro:arg name="laser_3d_secondary_enabled"    default="$(optenv HUSKY_LASER_3D_SECONDARY_ENABLED 0)" />
@@ -79,5 +87,5 @@
   <xacro:property name="realsense_model"          value="$(arg realsense_model)"/>
   <!-- Realsense Camera New -->
-  <xacro:arg name="realsense_enabled_new"             default="$(optenv HUSKY_REALSENSE_ENABLED 0)" />
+  <!-- <xacro:arg name="realsense_enabled_new"             default="$(optenv HUSKY_REALSENSE_ENABLED 1)" />
   <xacro:arg name="realsense_mode_new"               default="$(optenv HUSKY_REALSENSE_MODEL d435)"/>
   <xacro:arg name="realsense_topic_new"               default="$(optenv HUSKY_REALSENSE_TOPIC realsense)" />
@@ -85,4 +93,13 @@
   <xacro:arg name="realsense_parent_new"              default="$(optenv HUSKY_REALSENSE_PARENT top_plate_link)" />
   <xacro:arg name="realsense_xyz_new"                 default="$(optenv HUSKY_REALSENSE_XYZ 0.35 0 0.01)" />
+  <xacro:arg name="realsense_rpy_new"                 default="$(optenv HUSKY_REALSENSE_RPY 0 0 0)" />
+  <xacro:property name="realsense_model"          value="$(arg realsense_model)"/> -->
+  <!-- Realsense Camera New -->
+  <xacro:arg name="realsense_enabled_new"             default="$(optenv HUSKY_REALSENSE_ENABLED 1)" />
+  <xacro:arg name="realsense_mode_new"               default="$(optenv HUSKY_REALSENSE_MODEL d435)"/>
+  <xacro:arg name="realsense_topic_new"               default="$(optenv HUSKY_REALSENSE_TOPIC realsense)" />
+  <xacro:arg name="realsense_prefix_new"              default="$(optenv HUSKY_REALSENSE_PREFIX realsense_camera)" />
+  <xacro:arg name="realsense_parent_new"              default="$(optenv HUSKY_REALSENSE_PARENT base_link)" />
+  <xacro:arg name="realsense_xyz_new"                 default="$(optenv HUSKY_REALSENSE_XYZ 0.38502 0.0 0.31605)" />
   <xacro:arg name="realsense_rpy_new"                 default="$(optenv HUSKY_REALSENSE_RPY 0 0 0)" />
   <xacro:property name="realsense_model"          value="$(arg realsense_model)"/>
@@ -131,8 +148,9 @@
   <!-- <xacro:include filename="$(find husky_description)/urdf/accessories/flir_blackfly_mount.urdf.xacro"/> -->
   <!-- <xacro:include filename="$(find husky_description)/urdf/accessories/sensor_arch.urdf.xacro"/> -->
-  <!-- <xacro:include filename="$(find husky_description)/urdf/accessories/vlp16_mount.urdf.xacro"/> -->
+  <xacro:include filename="$(find husky_description)/urdf/accessories/vlp16_mount.urdf.xacro"/>
   <xacro:include filename="$(find husky_description)/urdf/decorations.urdf.xacro" />
   <xacro:include filename="$(find husky_description)/urdf/wheel.urdf.xacro" />
-  <xacro:include filename="$(find cpr_onav_description)/urdf/husky_observer.urdf.xacro" />
+  <xacro:include filename="$(find husky_description)/urdf/accessories/gnss_antenna.urdf.xacro" />
+  <xacro:include filename="$(find husky_description)/urdf/husky_observer.urdf.xacro" />
   <xacro:property name="M_PI" value="3.14159"/>
   <!-- Base Size -->
@@ -386,4 +404,16 @@
     </plugin>
   </gazebo>
+  <xacro:gnss_antenna
+      parent="base_link"
+      name="gps_left"
+      gps_num="1">
+    <origin xyz="-0.25814 0.35027 0.92479" rpy="0 0 0" />
+  </xacro:gnss_antenna>
+  <xacro:gnss_antenna
+      parent="base_link"
+      name="gps_right"
+      gps_num="2">
+    <origin xyz="-0.25814 -0.35027 0.92479" rpy="0 0 0" />
+  </xacro:gnss_antenna>
   <!-- Optional custom includes. -->
   <xacro:include filename="$(arg urdf_extras)" />

Commit message: feat: add IMU noise profiles and configurable parameters for benchmarking and simulation

File: husky_description/urdf/husky.urdf.xacro (robot description, xacro)
@@ -26,11 +26,11 @@
   <xacro:arg name="imu_rpy"     default="$(optenv HUSKY_IMU_RPY 0 -1.5708 3.1416)"/>
   <xacro:arg name="imu_parent"  default="$(optenv HUSKY_IMU_PARENT base_link)"/>
-  <!-- IMU noise parameters (configurable via env vars for benchmarking) -->
-  <xacro:arg name="imu_accel_drift"     default="$(optenv HUSKY_IMU_ACCEL_DRIFT 0.005)"/>
-  <xacro:arg name="imu_accel_noise"     default="$(optenv HUSKY_IMU_ACCEL_NOISE 0.005)"/>
-  <xacro:arg name="imu_rate_drift"      default="$(optenv HUSKY_IMU_RATE_DRIFT 0.005)"/>
-  <xacro:arg name="imu_rate_noise"      default="$(optenv HUSKY_IMU_RATE_NOISE 0.005)"/>
-  <xacro:arg name="imu_heading_drift"   default="$(optenv HUSKY_IMU_HEADING_DRIFT 0.005)"/>
-  <xacro:arg name="imu_heading_noise"   default="$(optenv HUSKY_IMU_HEADING_NOISE 0.005)"/>
+  <!-- IMU noise profile (highend/mid/lowend) loaded from config/imu_profiles.yaml.
+       Select via `imu_profile:=<name>` launch arg or HUSKY_IMU_PROFILE env var. -->
+  <xacro:arg name="imu_profile" default="$(optenv HUSKY_IMU_PROFILE mid)"/>
+  <xacro:property name="imu_profile_name" value="$(arg imu_profile)"/>
+  <xacro:property name="imu_profiles_path" value="$(find husky_description)/config/imu_profiles.yaml"/>
+  <xacro:property name="imu_profiles" value="${xacro.load_yaml(imu_profiles_path)}"/>
+  <xacro:property name="imu_cfg" value="${imu_profiles[imu_profile_name]}"/>
   <!-- LMS1XX Laser Primary and Secondary -->
   <xacro:arg name="laser_enabled"           default="$(optenv HUSKY_LMS1XX_ENABLED 0)" />
@@ -388,10 +388,10 @@
       <bodyName>base_link</bodyName>
       <topicName>imu/data</topicName>
-      <accelDrift>$(arg imu_accel_drift) $(arg imu_accel_drift) $(arg imu_accel_drift)</accelDrift>
-      <accelGaussianNoise>$(arg imu_accel_noise) $(arg imu_accel_noise) $(arg imu_accel_noise)</accelGaussianNoise>
-      <rateDrift>$(arg imu_rate_drift) $(arg imu_rate_drift) $(arg imu_rate_drift)</rateDrift>
-      <rateGaussianNoise>$(arg imu_rate_noise) $(arg imu_rate_noise) $(arg imu_rate_noise)</rateGaussianNoise>
-      <headingDrift>$(arg imu_heading_drift)</headingDrift>
-      <headingGaussianNoise>$(arg imu_heading_noise)</headingGaussianNoise>
+      <accelDrift>${imu_cfg['accel_drift']} ${imu_cfg['accel_drift']} ${imu_cfg['accel_drift']}</accelDrift>
+      <accelGaussianNoise>${imu_cfg['accel_noise']} ${imu_cfg['accel_noise']} ${imu_cfg['accel_noise']}</accelGaussianNoise>
+      <rateDrift>${imu_cfg['rate_drift']} ${imu_cfg['rate_drift']} ${imu_cfg['rate_drift']}</rateDrift>
+      <rateGaussianNoise>${imu_cfg['rate_noise']} ${imu_cfg['rate_noise']} ${imu_cfg['rate_noise']}</rateGaussianNoise>
+      <headingDrift>${imu_cfg['heading_drift']}</headingDrift>
+      <headingGaussianNoise>${imu_cfg['heading_noise']}</headingGaussianNoise>
     </plugin>
   </gazebo>
