Commit message: feat: made changes to gnss antenna urdf to publish diff gps points for left and right and then calc heading

File: husky_description/urdf/accessories/gnss_antenna.urdf.xacro (robot description, xacro)
@@ -18,8 +18,16 @@
         <origin xyz="0 0 ${0.065/2}" rpy="0 0 0" />
       </collision>
+      <inertial>
+        <mass value="0.1"/>   <!-- very small mass (for revolute joints inertial mas needed) -->
+        <origin xyz="0 0 0" rpy="0 0 0"/>
+        <inertia ixx="1e-5" iyy="1e-5" izz="1e-5" ixy="0" ixz="0" iyz="0"/>
+      </inertial>
     </link>
-    <joint name="${name}_joint" type="fixed">
+    <joint name="${name}_joint" type="revolute">  <!-- changed fixed to revolute publish different gps points -->
       <parent link="${parent}" />
       <child link="${name}_link" />
+      <axis xyz="0 0 1" />  <!-- Required for revolute -->
+      <limit lower="0" upper="0" effort="0.1" velocity="0.1"/>
+      <dynamics damping="0.1" friction="0.1"/>
       <xacro:insert_block name="origin" />
     </joint>
